Commit message: Making sim same as real bot

File: description/robot_core.xacro (robot description, xacro)
@@ -19,18 +19,18 @@
         <parent link="base_link"/>
         <child link="chassis"/>
-        <origin xyz="-0.1 0 0"/>
+        <origin xyz="-0.05 0 0"/>
     </joint>
     <link name="chassis">
         <visual>
-            <origin xyz="0.15 0 0.05" rpy="0 0 ${pi/2}"/>
+            <origin xyz="0.15 0 0.005" rpy="0 0 ${pi/2}"/>
             <geometry>
-                <box size="0.3 0.3 0.15"/>
+                <box size="0.21 0.265 0.005"/>
             </geometry>
             <material name="fontys_purple"/>
         </visual>
         <collision>
-            <origin xyz="0.15 0 0.075"/>
+            <origin xyz="0.15 0 0.005"/>
             <geometry>
-                <box size="0.3 0.3 0.15"/>
+                <box size="0.21 0.265 0.005"/>
             </geometry>
         </collision>
@@ -40,5 +40,5 @@
     </link>
     <gazebo reference="chassis">
-        <material>Gazebo/Purple</material>
+        <material>Gazebo/Black</material>
     </gazebo>
     <!-- LEFT WHEEL LINK -->
@@ -46,5 +46,5 @@
         <parent link="base_link"/>
         <child link="left_wheel"/>
-        <origin xyz="0 0.175 0" rpy="-${pi/2} 0 0" />
+        <origin xyz="0 0.115 0" rpy="-${pi/2} 0 0" />
         <axis xyz="0 0 1"/>
     </joint>
@@ -52,5 +52,5 @@
         <visual>
             <geometry>
-                <cylinder radius="0.05" length="0.04"/>
+                <cylinder radius="0.025" length="0.015"/>
             </geometry>
             <material name="black"/>
@@ -58,5 +58,5 @@
         <collision>
             <geometry>
-                <cylinder radius="0.05" length="0.04"/>
+                <cylinder radius="0.025" length="0.015"/>
             </geometry>
         </collision>
@@ -66,5 +66,5 @@
     </link>
     <gazebo reference="left_wheel">
-        <material>Gazebo/Black</material>
+        <material>Gazebo/Yellow</material>
     </gazebo>
     <!-- RIGHT WHEEL LINK -->
@@ -72,5 +72,5 @@
         <parent link="base_link"/>
         <child link="right_wheel"/>
-        <origin xyz="0 -0.175 0" rpy="${pi/2} 0 0" />
+        <origin xyz="0 -0.115 0" rpy="${pi/2} 0 0" />
         <axis xyz="0 0 -1"/>
     </joint>
@@ -78,5 +78,5 @@
         <visual>
             <geometry>
-                <cylinder radius="0.05" length="0.04"/>
+                <cylinder radius="0.025" length="0.015"/>
             </geometry>
             <material name="black"/>
@@ -84,5 +84,5 @@
         <collision>
             <geometry>
-                <cylinder radius="0.05" length="0.04"/>
+                <cylinder radius="0.025" length="0.015"/>
             </geometry>
         </collision>
@@ -92,5 +92,5 @@
     </link>
     <gazebo reference="right_wheel">
-        <material>Gazebo/Black</material>
+        <material>Gazebo/Yellow</material>
     </gazebo>
     <!-- CASTER WHEEL LINK -->
@@ -98,10 +98,10 @@
         <parent link="chassis"/>
         <child link="caster_wheel"/>
-        <origin xyz="0.24 0 0"/>
+        <origin xyz="0.26 0 0"/>
     </joint>
     <link name="caster_wheel">
         <visual>
             <geometry>
-                <sphere radius="0.05"/>
+                <sphere radius="0.025"/>
             </geometry>
             <material name="grey"/>
@@ -109,5 +109,5 @@
         <collision>
             <geometry>
-                <sphere radius="0.05"/>
+                <sphere radius="0.025"/>
             </geometry>
         </collision>
@@ -117,5 +117,5 @@
     </link>
     <gazebo reference="caster_wheel">
-        <material>Gazebo/Grey</material>
+        <material>Gazebo/White</material>
         <mu1 value="0.001"/> <!-- friction -->
         <mu2 value="0.001"/>
